Commit message: create rviz.launch

File: urdf/spiderrobot.xacro (robot description, xacro)
@@ -4,4 +4,5 @@
 <xacro:include filename="$(find robot_contest)/urdf/spiderrobot.trans" />
 <xacro:include filename="$(find robot_contest)/urdf/spiderrobot.gazebo" />
+<link name="dummy"></link>
 <link name="base_link">
   <inertial>
@@ -1004,4 +1005,8 @@
   </collision>
 </link>
+<joint name="dummy_joint" type="fixed">
+  <parent link="dummy"/>
+  <child link="base_link"/>
+</joint>
 <joint name="fixed1" type="fixed">
   <origin xyz="0.137126 0.047626 0.0015" rpy="0 0 0"/>
