Commit message: change model

File: urdf/spider_robot.xacro (robot description, xacro)
@@ -6,771 +6,886 @@
 <link name="dummy">
 </link>
-<link name="base_link">
-  <inertial>
-    <origin xyz="0.012498209191529774 1.7496974071002831e-13 0.0009731404762877922" rpy="0 0 0"/>
-    <mass value="1.80778160581464"/>
-    <inertia ixx="0.027407" iyy="0.010993" izz="0.028617" ixy="-0.0" iyz="0.0" ixz="0.002015"/>
-  </inertial>
-  <visual>
-    <origin xyz="0 0 0" rpy="0 0 0"/>
-    <geometry>
-      <mesh filename="package://robot_contest/meshes/base_link.stl" scale="0.001 0.001 0.001"/>
-    </geometry>
-    <material name="_"/>
-  </visual>
-  <collision>
-    <origin xyz="0 0 0" rpy="0 0 0"/>
-    <geometry>
-      <mesh filename="package://robot_contest/meshes/base_link.stl" scale="0.001 0.001 0.001"/>
-    </geometry>
-  </collision>
-</link>
-<link name="part1_1">
-  <inertial>
-    <origin xyz="0.0406275735859281 0.07461587091689897 0.011754836260053298" rpy="0 0 0"/>
-    <mass value="0.0413494129978488"/>
-    <inertia ixx="0.000354" iyy="5.1e-05" izz="0.000367" ixy="-8.6e-05" iyz="3.2e-05" ixz="1e-05"/>
-  </inertial>
-  <visual>
-    <origin xyz="-0.067071 0.156571 -0.0" rpy="0 0 0"/>
-    <geometry>
-      <mesh filename="package://robot_contest/meshes/part1_1.stl" scale="0.001 0.001 0.001"/>
-    </geometry>
-    <material name="_"/>
-  </visual>
-  <collision>
-    <origin xyz="-0.067071 0.156571 -0.0" rpy="0 0 0"/>
-    <geometry>
-      <mesh filename="package://robot_contest/meshes/part1_1.stl" scale="0.001 0.001 0.001"/>
-    </geometry>
-  </collision>
-</link>
-<link name="part2_1">
-  <inertial>
-    <origin xyz="0.093210203534517 0.1995912315229256 -0.014453508806619629" rpy="0 0 0"/>
-    <mass value="0.531782740534772"/>
-    <inertia ixx="0.009933" iyy="0.000995" izz="0.010806" ixy="-0.001933" iyz="0.000632" ixz="0.000138"/>
-  </inertial>
-  <visual>
-    <origin xyz="-0.082009 0.208101 -0.020875" rpy="0 0 0"/>
-    <geometry>
-      <mesh filename="package://robot_contest/meshes/part2_1.stl" scale="0.001 0.001 0.001"/>
-    </geometry>
-    <material name="_"/>
-  </visual>
-  <collision>
-    <origin xyz="-0.082009 0.208101 -0.020875" rpy="0 0 0"/>
-    <geometry>
-      <mesh filename="package://robot_contest/meshes/part2_1.stl" scale="0.001 0.001 0.001"/>
-    </geometry>
-  </collision>
-</link>
-<link name="part3_1">
-  <inertial>
-    <origin xyz="0.020802990843692082 0.10926815025858176 -0.005288903492875214" rpy="0 0 0"/>
-    <mass value="0.12505650813053104"/>
-    <inertia ixx="0.002641" iyy="0.000153" izz="0.002722" ixy="-0.000128" iyz="0.000259" ixz="1.5e-05"/>
-  </inertial>
-  <visual>
-    <origin xyz="-0.173452 0.231662 -0.020875" rpy="0 0 0"/>
-    <geometry>
-      <mesh filename="package://robot_contest/meshes/part3_1.stl" scale="0.001 0.001 0.001"/>
-    </geometry>
-    <material name="_"/>
-  </visual>
-  <collision>
-    <origin xyz="-0.173452 0.231662 -0.020875" rpy="0 0 0"/>
-    <geometry>
-      <mesh filename="package://robot_contest/meshes/part3_1.stl" scale="0.001 0.001 0.001"/>
-    </geometry>
-  </collision>
-</link>
-<link name="d_part1_1">
-  <inertial>
-    <origin xyz="-1.5718367696315738e-07 -7.586335737386207e-08 7.494005416219807e-16" rpy="0 0 0"/>
-    <mass value="4.110250388446646e-06"/>
-    <inertia ixx="0.0" iyy="0.0" izz="0.0" ixy="0.0" iyz="0.0" ixz="0.0"/>
-  </inertial>
-  <visual>
-    <origin xyz="-0.257686 0.345418 -0.020875" rpy="0 0 0"/>
-    <geometry>
-      <mesh filename="package://robot_contest/meshes/d_part1_1.stl" scale="0.001 0.001 0.001"/>
-    </geometry>
-    <material name="_"/>
-  </visual>
-  <collision>
-    <origin xyz="-0.257686 0.345418 -0.020875" rpy="0 0 0"/>
-    <geometry>
-      <mesh filename="package://robot_contest/meshes/d_part1_1.stl" scale="0.001 0.001 0.001"/>
-    </geometry>
-  </collision>
-</link>
-<link name="d_part2_1">
-  <inertial>
-    <origin xyz="-1.5718367696315738e-07 -7.586335737386207e-08 7.494005416219807e-16" rpy="0 0 0"/>
-    <mass value="4.110250388446646e-06"/>
-    <inertia ixx="0.0" iyy="0.0" izz="0.0" ixy="0.0" iyz="0.0" ixz="0.0"/>
-  </inertial>
-  <visual>
-    <origin xyz="-0.257686 0.345418 -0.020875" rpy="0 0 0"/>
-    <geometry>
-      <mesh filename="package://robot_contest/meshes/d_part2_1.stl" scale="0.001 0.001 0.001"/>
-    </geometry>
-    <material name="_"/>
-  </visual>
-  <collision>
-    <origin xyz="-0.257686 0.345418 -0.020875" rpy="0 0 0"/>
-    <geometry>
-      <mesh filename="package://robot_contest/meshes/d_part2_1.stl" scale="0.001 0.001 0.001"/>
-    </geometry>
-  </collision>
-</link>
-<link name="d_part3_1">
-  <inertial>
-    <origin xyz="-1.5718367696315738e-07 -7.586335737386207e-08 7.424616477180734e-16" rpy="0 0 0"/>
-    <mass value="4.110250388446646e-06"/>
-    <inertia ixx="0.0" iyy="0.0" izz="0.0" ixy="0.0" iyz="0.0" ixz="-0.0"/>
-  </inertial>
-  <visual>
-    <origin xyz="-0.257686 0.345418 -0.020875" rpy="0 0 0"/>
-    <geometry>
-      <mesh filename="package://robot_contest/meshes/d_part3_1.stl" scale="0.001 0.001 0.001"/>
-    </geometry>
-    <material name="_"/>
-  </visual>
-  <collision>
-    <origin xyz="-0.257686 0.345418 -0.020875" rpy="0 0 0"/>
-    <geometry>
-      <mesh filename="package://robot_contest/meshes/d_part3_1.stl" scale="0.001 0.001 0.001"/>
-    </geometry>
-  </collision>
-</link>
-<link name="part4_1">
-  <inertial>
-    <origin xyz="-0.07691919454265221 0.007217146282982756 0.008868255825853702" rpy="0 0 0"/>
-    <mass value="0.0413494129978488"/>
-    <inertia ixx="5.8e-05" iyy="0.000171" izz="0.000186" ixy="5.7e-05" iyz="1.1e-05" ixz="-2.6e-05"/>
-  </inertial>
-  <visual>
-    <origin xyz="0.067071 0.156571 0.0" rpy="0 0 0"/>
-    <geometry>
-      <mesh filename="package://robot_contest/meshes/part4_1.stl" scale="0.001 0.001 0.001"/>
-    </geometry>
-    <material name="_"/>
-  </visual>
-  <collision>
-    <origin xyz="0.067071 0.156571 0.0" rpy="0 0 0"/>
-    <geometry>
-      <mesh filename="package://robot_contest/meshes/part4_1.stl" scale="0.001 0.001 0.001"/>
-    </geometry>
-  </collision>
-</link>
-<link name="part5_1">
-  <inertial>
-    <origin xyz="0.06214795924517012 -0.07868893741539248 -0.01445350881492818" rpy="0 0 0"/>
-    <mass value="0.531782740534772"/>
-    <inertia ixx="0.001749" iyy="0.003068" izz="0.004695" ixy="0.001505" iyz="-0.000207" ixz="0.000331"/>
-  </inertial>
-  <visual>
-    <origin xyz="0.082009 0.208101 -0.020875" rpy="0 0 0"/>
-    <geometry>
-      <mesh filename="package://robot_contest/meshes/part5_1.stl" scale="0.001 0.001 0.001"/>
-    </geometry>
-    <material name="_"/>
-  </visual>
-  <collision>
-    <origin xyz="0.082009 0.208101 -0.020875" rpy="0 0 0"/>
-    <geometry>
-      <mesh filename="package://robot_contest/meshes/part5_1.stl" scale="0.001 0.001 0.001"/>
-    </geometry>
-  </collision>
-</link>
-<link name="part6_1">
-  <inertial>
-    <origin xyz="-0.03147293086420935 0.10321299484181759 -0.005288903492875221" rpy="0 0 0"/>
-    <mass value="0.12505650813053248"/>
-    <inertia ixx="0.002441" iyy="0.000189" izz="0.002558" ixy="0.000319" iyz="0.000242" ixz="-3.3e-05"/>
-  </inertial>
-  <visual>
-    <origin xyz="0.173452 0.231662 -0.020875" rpy="0 0 0"/>
-    <geometry>
-      <mesh filename="package://robot_contest/meshes/part6_1.stl" scale="0.001 0.001 0.001"/>
-    </geometry>
-    <material name="_"/>
-  </visual>
-  <collision>
-    <origin xyz="0.173452 0.231662 -0.020875" rpy="0 0 0"/>
-    <geometry>
-      <mesh filename="package://robot_contest/meshes/part6_1.stl" scale="0.001 0.001 0.001"/>
-    </geometry>
-  </collision>
-</link>
-<link name="d_part4_1">
-  <inertial>
-    <origin xyz="1.571836772962243e-07 -7.586335737386207e-08 9.54097911787244e-16" rpy="0 0 0"/>
-    <mass value="4.110250388446646e-06"/>
-    <inertia ixx="0.0" iyy="0.0" izz="0.0" ixy="0.0" iyz="-0.0" ixz="-0.0"/>
-  </inertial>
-  <visual>
-    <origin xyz="0.257686 0.345418 -0.020875" rpy="0 0 0"/>
-    <geometry>
-      <mesh filename="package://robot_contest/meshes/d_part4_1.stl" scale="0.001 0.001 0.001"/>
-    </geometry>
-    <material name="_"/>
-  </visual>
-  <collision>
-    <origin xyz="0.257686 0.345418 -0.020875" rpy="0 0 0"/>
-    <geometry>
-      <mesh filename="package://robot_contest/meshes/d_part4_1.stl" scale="0.001 0.001 0.001"/>
-    </geometry>
-  </collision>
-</link>
-<link name="d_part5_1">
-  <inertial>
-    <origin xyz="1.571836772962243e-07 -7.586335737386207e-08 9.54097911787244e-16" rpy="0 0 0"/>
-    <mass value="4.110250388446646e-06"/>
-    <inertia ixx="0.0" iyy="0.0" izz="0.0" ixy="0.0" iyz="-0.0" ixz="-0.0"/>
-  </inertial>
-  <visual>
-    <origin xyz="0.257686 0.345418 -0.020875" rpy="0 0 0"/>
-    <geometry>
-      <mesh filename="package://robot_contest/meshes/d_part5_1.stl" scale="0.001 0.001 0.001"/>
-    </geometry>
-    <material name="_"/>
-  </visual>
-  <collision>
-    <origin xyz="0.257686 0.345418 -0.020875" rpy="0 0 0"/>
-    <geometry>
-      <mesh filename="package://robot_contest/meshes/d_part5_1.stl" scale="0.001 0.001 0.001"/>
-    </geometry>
-  </collision>
-</link>
-<link name="d_part6_1">
-  <inertial>
-    <origin xyz="1.571836772962243e-07 -7.586335737386207e-08 2.42861286636753e-16" rpy="0 0 0"/>
-    <mass value="4.110250388446646e-06"/>
-    <inertia ixx="0.0" iyy="0.0" izz="0.0" ixy="-0.0" iyz="0.0" ixz="0.0"/>
-  </inertial>
-  <visual>
-    <origin xyz="0.257686 0.345418 -0.020875" rpy="0 0 0"/>
-    <geometry>
-      <mesh filename="package://robot_contest/meshes/d_part6_1.stl" scale="0.001 0.001 0.001"/>
-    </geometry>
-    <material name="_"/>
-  </visual>
-  <collision>
-    <origin xyz="0.257686 0.345418 -0.020875" rpy="0 0 0"/>
-    <geometry>
-      <mesh filename="package://robot_contest/meshes/d_part6_1.stl" scale="0.001 0.001 0.001"/>
-    </geometry>
-  </collision>
-</link>
-<link name="part7_1">
-  <inertial>
-    <origin xyz="0.04760800534982393 0.0014432902170995274 0.011754836260053147" rpy="0 0 0"/>
-    <mass value="0.0413494129978488"/>
-    <inertia ixx="3.5e-05" iyy="5e-05" izz="4.7e-05" ixy="-3e-06" iyz="1e-06" ixz="1e-05"/>
-  </inertial>
-  <visual>
-    <origin xyz="-0.09 -0.0 -0.0" rpy="0 0 0"/>
-    <geometry>
-      <mesh filename="package://robot_contest/meshes/part7_1.stl" scale="0.001 0.001 0.001"/>
-    </geometry>
-    <material name="_"/>
-  </visual>
-  <collision>
-    <origin xyz="-0.09 -0.0 -0.0" rpy="0 0 0"/>
-    <geometry>
-      <mesh filename="package://robot_contest/meshes/part7_1.stl" scale="0.001 0.001 0.001"/>
-    </geometry>
-  </collision>
-</link>
-<link name="part8_1">
-  <inertial>
-    <origin xyz="0.09488310137697165 0.0790088049554718 -0.014453508806619749" rpy="0 0 0"/>
-    <mass value="0.531782740534772"/>
-    <inertia ixx="0.001274" iyy="0.001239" izz="0.002391" ixy="-0.000593" iyz="0.000158" ixz="0.000164"/>
-  </inertial>
-  <visual>
-    <origin xyz="-0.137 0.025875 -0.020875" rpy="0 0 0"/>
-    <geometry>
-      <mesh filename="package://robot_contest/meshes/part8_1.stl" scale="0.001 0.001 0.001"/>
-    </geometry>
-    <material name="_"/>
-  </visual>
-  <collision>
-    <origin xyz="-0.137 0.025875 -0.020875" rpy="0 0 0"/>
-    <geometry>
-      <mesh filename="package://robot_contest/meshes/part8_1.stl" scale="0.001 0.001 0.001"/>
-    </geometry>
-  </collision>
-</link>
-<link name="part9_1">
-  <inertial>
-    <origin xyz="0.08291366552091187 -0.014833512817442334 -0.005288903492875382" rpy="0 0 0"/>
-    <mass value="0.12505650813053104"/>
-    <inertia ixx="8.9e-05" iyy="0.000408" izz="0.000425" ixy="-1.9e-05" iyz="1.4e-05" ixz="7.7e-05"/>
-  </inertial>
-  <visual>
-    <origin xyz="-0.21832 -0.022125 -0.020875" rpy="0 0 0"/>
-    <geometry>
-      <mesh filename="package://robot_contest/meshes/part9_1.stl" scale="0.001 0.001 0.001"/>
-    </geometry>
-    <material name="_"/>
-  </visual>
-  <collision>
-    <origin xyz="-0.21832 -0.022125 -0.020875" rpy="0 0 0"/>
-    <geometry>
-      <mesh filename="package://robot_contest/meshes/part9_1.stl" scale="0.001 0.001 0.001"/>
-    </geometry>
-  </collision>
-</link>
-<link name="d_part7_1">
-  <inertial>
-    <origin xyz="4.996003610813204e-16 -2.985892783025079e-16 3.7470027081099033e-16" rpy="0 0 0"/>
-    <mass value="4.110250388446646e-06"/>
-    <inertia ixx="0.0" iyy="0.0" izz="0.0" ixy="0.0" iyz="0.0" ixz="0.0"/>
-  </inertial>
-  <visual>
-    <origin xyz="-0.35832 -0.00125 -0.020875" rpy="0 0 0"/>
-    <geometry>
-      <mesh filename="package://robot_contest/meshes/d_part7_1.stl" scale="0.001 0.001 0.001"/>
-    </geometry>
-    <material name="_"/>
-  </visual>
-  <collision>
-    <origin xyz="-0.35832 -0.00125 -0.020875" rpy="0 0 0"/>
-    <geometry>
-      <mesh filename="package://robot_contest/meshes/d_part7_1.stl" scale="0.001 0.001 0.001"/>
-    </geometry>
-  </collision>
-</link>
-<link name="d_part8_1">
-  <inertial>
-    <origin xyz="4.996003610813204e-16 -2.985892783025079e-16 3.7470027081099033e-16" rpy="0 0 0"/>
-    <mass value="4.110250388446646e-06"/>
-    <inertia ixx="0.0" iyy="0.0" izz="0.0" ixy="0.0" iyz="0.0" ixz="0.0"/>
-  </inertial>
-  <visual>
-    <origin xyz="-0.35832 -0.00125 -0.020875" rpy="0 0 0"/>
-    <geometry>
-      <mesh filename="package://robot_contest/meshes/d_part8_1.stl" scale="0.001 0.001 0.001"/>
-    </geometry>
-    <material name="_"/>
-  </visual>
-  <collision>
-    <origin xyz="-0.35832 -0.00125 -0.020875" rpy="0 0 0"/>
-    <geometry>
-      <mesh filename="package://robot_contest/meshes/d_part8_1.stl" scale="0.001 0.001 0.001"/>
-    </geometry>
-  </collision>
-</link>
-<link name="d_part9_1">
-  <inertial>
-    <origin xyz="4.996003610813204e-16 -2.985892783025079e-16 3.7470027081099033e-16" rpy="0 0 0"/>
-    <mass value="4.110250388446646e-06"/>
-    <inertia ixx="0.0" iyy="0.0" izz="0.0" ixy="0.0" iyz="0.0" ixz="0.0"/>
-  </inertial>
-  <visual>
-    <origin xyz="-0.35832 -0.00125 -0.020875" rpy="0 0 0"/>
-    <geometry>
-      <mesh filename="package://robot_contest/meshes/d_part9_1.stl" scale="0.001 0.001 0.001"/>
-    </geometry>
-    <material name="_"/>
-  </visual>
-  <collision>
-    <origin xyz="-0.35832 -0.00125 -0.020875" rpy="0 0 0"/>
-    <geometry>
-      <mesh filename="package://robot_contest/meshes/d_part9_1.stl" scale="0.001 0.001 0.001"/>
-    </geometry>
-  </collision>
-</link>
-<link name="part10_1">
-  <inertial>
-    <origin xyz="-0.0683460744679519 0.0014432902170994414 0.00886825582585395" rpy="0 0 0"/>
-    <mass value="0.0413494129978488"/>
-    <inertia ixx="3.7e-05" iyy="0.000108" izz="0.000102" ixy="4e-06" iyz="1e-06" ixz="-1.9e-05"/>
-  </inertial>
-  <visual>
-    <origin xyz="0.09 -0.0 0.0" rpy="0 0 0"/>
-    <geometry>
-      <mesh filename="package://robot_contest/meshes/part10_1.stl" scale="0.001 0.001 0.001"/>
-    </geometry>
-    <material name="_"/>
-  </visual>
-  <collision>
-    <origin xyz="0.09 -0.0 0.0" rpy="0 0 0"/>
-    <geometry>
-      <mesh filename="package://robot_contest/meshes/part10_1.stl" scale="0.001 0.001 0.001"/>
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