Commit message: fix model

File: urdf/spider_robot.xacro (robot description, xacro)
@@ -1,7 +1,7 @@
 <?xml version="1.0" ?>
 <robot name="spider_robot" xmlns:xacro="http://www.ros.org/wiki/xacro">
-<xacro:include filename="$(find robot_contest)/urdf/materials.xacro" />
-<xacro:include filename="$(find robot_contest)/urdf/spider_robot.trans" />
-<xacro:include filename="$(find robot_contest)/urdf/spider_robot.gazebo" />
+<xacro:include filename="$(find spider_robot_description)/urdf/materials.xacro" />
+<xacro:include filename="$(find spider_robot_description)/urdf/spider_robot.trans" />
+<xacro:include filename="$(find spider_robot_description)/urdf/spider_robot.gazebo" />
 <link name="dummy">
 </link>
@@ -19,5 +19,5 @@
     <origin xyz="0 0 0" rpy="0 0 0"/>
     <geometry>
-      <mesh filename="package://robot_contest/meshes/base_link.stl" scale="0.001 0.001 0.001"/>
+      <mesh filename="package://spider_robot_description/meshes/base_link.stl" scale="0.001 0.001 0.001"/>
     </geometry>
     <material name="_"/>
@@ -26,5 +26,5 @@
     <origin xyz="0 0 0" rpy="0 0 0"/>
     <geometry>
-      <mesh filename="package://robot_contest/meshes/base_link.stl" scale="0.001 0.001 0.001"/>
+      <mesh filename="package://spider_robot_description/meshes/base_link.stl" scale="0.001 0.001 0.001"/>
     </geometry>
   </collision>
@@ -39,5 +39,5 @@
     <origin xyz="-0.095 -0.0545 -0.005" rpy="0 0 0"/>
     <geometry>
-      <mesh filename="package://robot_contest/meshes/part1_1.stl" scale="0.001 0.001 0.001"/>
+      <mesh filename="package://spider_robot_description/meshes/part1_1.stl" scale="0.001 0.001 0.001"/>
     </geometry>
     <material name="_"/>
@@ -46,5 +46,5 @@
     <origin xyz="-0.095 -0.0545 -0.005" rpy="0 0 0"/>
     <geometry>
-      <mesh filename="package://robot_contest/meshes/part1_1.stl" scale="0.001 0.001 0.001"/>
+      <mesh filename="package://spider_robot_description/meshes/part1_1.stl" scale="0.001 0.001 0.001"/>
     </geometry>
   </collision>
@@ -59,5 +59,5 @@
     <origin xyz="-0.12058 -0.116673 -0.0304" rpy="0 0 0"/>
     <geometry>
-      <mesh filename="package://robot_contest/meshes/part2_1.stl" scale="0.001 0.001 0.001"/>
+      <mesh filename="package://spider_robot_description/meshes/part2_1.stl" scale="0.001 0.001 0.001"/>
     </geometry>
     <material name="_"/>
@@ -66,5 +66,5 @@
     <origin xyz="-0.12058 -0.116673 -0.0304" rpy="0 0 0"/>
     <geometry>
-      <mesh filename="package://robot_contest/meshes/part2_1.stl" scale="0.001 0.001 0.001"/>
+      <mesh filename="package://spider_robot_description/meshes/part2_1.stl" scale="0.001 0.001 0.001"/>
     </geometry>
   </collision>
@@ -79,5 +79,5 @@
     <origin xyz="-0.095 0.0545 -0.005" rpy="0 0 0"/>
     <geometry>
-      <mesh filename="package://robot_contest/meshes/part4_1.stl" scale="0.001 0.001 0.001"/>
+      <mesh filename="package://spider_robot_description/meshes/part4_1.stl" scale="0.001 0.001 0.001"/>
     </geometry>
     <material name="_"/>
@@ -86,5 +86,5 @@
     <origin xyz="-0.095 0.0545 -0.005" rpy="0 0 0"/>
     <geometry>
-      <mesh filename="package://robot_contest/meshes/part4_1.stl" scale="0.001 0.001 0.001"/>
+      <mesh filename="package://spider_robot_description/meshes/part4_1.stl" scale="0.001 0.001 0.001"/>
     </geometry>
   </collision>
@@ -99,5 +99,5 @@
     <origin xyz="-0.12058 0.116673 -0.0304" rpy="0 0 0"/>
     <geometry>
-      <mesh filename="package://robot_contest/meshes/part5_1.stl" scale="0.001 0.001 0.001"/>
+      <mesh filename="package://spider_robot_description/meshes/part5_1.stl" scale="0.001 0.001 0.001"/>
     </geometry>
     <material name="_"/>
@@ -106,5 +106,5 @@
     <origin xyz="-0.12058 0.116673 -0.0304" rpy="0 0 0"/>
     <geometry>
-      <mesh filename="package://robot_contest/meshes/part5_1.stl" scale="0.001 0.001 0.001"/>
+      <mesh filename="package://spider_robot_description/meshes/part5_1.stl" scale="0.001 0.001 0.001"/>
     </geometry>
   </collision>
@@ -119,5 +119,5 @@
     <origin xyz="-0.0 -0.0545 -0.005" rpy="0 0 0"/>
     <geometry>
-      <mesh filename="package://robot_contest/meshes/part7_1.stl" scale="0.001 0.001 0.001"/>
+      <mesh filename="package://spider_robot_description/meshes/part7_1.stl" scale="0.001 0.001 0.001"/>
     </geometry>
     <material name="_"/>
@@ -126,5 +126,5 @@
     <origin xyz="-0.0 -0.0545 -0.005" rpy="0 0 0"/>
     <geometry>
-      <mesh filename="package://robot_contest/meshes/part7_1.stl" scale="0.001 0.001 0.001"/>
+      <mesh filename="package://spider_robot_description/meshes/part7_1.stl" scale="0.001 0.001 0.001"/>
     </geometry>
   </collision>
@@ -139,5 +139,5 @@
     <origin xyz="0.025875 -0.116551 -0.0304" rpy="0 0 0"/>
     <geometry>
-      <mesh filename="package://robot_contest/meshes/part8_1.stl" scale="0.001 0.001 0.001"/>
+      <mesh filename="package://spider_robot_description/meshes/part8_1.stl" scale="0.001 0.001 0.001"/>
     </geometry>
     <material name="_"/>
@@ -146,5 +146,5 @@
     <origin xyz="0.025875 -0.116551 -0.0304" rpy="0 0 0"/>
     <geometry>
-      <mesh filename="package://robot_contest/meshes/part8_1.stl" scale="0.001 0.001 0.001"/>
+      <mesh filename="package://spider_robot_description/meshes/part8_1.stl" scale="0.001 0.001 0.001"/>
     </geometry>
   </collision>
@@ -159,5 +159,5 @@
     <origin xyz="0.0 0.0545 -0.005" rpy="0 0 0"/>
     <geometry>
-      <mesh filename="package://robot_contest/meshes/part10_1.stl" scale="0.001 0.001 0.001"/>
+      <mesh filename="package://spider_robot_description/meshes/part10_1.stl" scale="0.001 0.001 0.001"/>
     </geometry>
     <material name="_"/>
@@ -166,5 +166,5 @@
     <origin xyz="0.0 0.0545 -0.005" rpy="0 0 0"/>
     <geometry>
-      <mesh filename="package://robot_contest/meshes/part10_1.stl" scale="0.001 0.001 0.001"/>
+      <mesh filename="package://spider_robot_description/meshes/part10_1.stl" scale="0.001 0.001 0.001"/>
     </geometry>
   </collision>
@@ -179,5 +179,5 @@
     <origin xyz="0.025875 0.116551 -0.0304" rpy="0 0 0"/>
     <geometry>
-      <mesh filename="package://robot_contest/meshes/part11_1.stl" scale="0.001 0.001 0.001"/>
+      <mesh filename="package://spider_robot_description/meshes/part11_1.stl" scale="0.001 0.001 0.001"/>
     </geometry>
     <material name="_"/>
@@ -186,5 +186,5 @@
     <origin xyz="0.025875 0.116551 -0.0304" rpy="0 0 0"/>
     <geometry>
-      <mesh filename="package://robot_contest/meshes/part11_1.stl" scale="0.001 0.001 0.001"/>
+      <mesh filename="package://spider_robot_description/meshes/part11_1.stl" scale="0.001 0.001 0.001"/>
     </geometry>
   </collision>
@@ -199,5 +199,5 @@
     <origin xyz="0.095 -0.0545 -0.005" rpy="0 0 0"/>
     <geometry>
-      <mesh filename="package://robot_contest/meshes/part13_1.stl" scale="0.001 0.001 0.001"/>
+      <mesh filename="package://spider_robot_description/meshes/part13_1.stl" scale="0.001 0.001 0.001"/>
     </geometry>
     <material name="_"/>
@@ -206,5 +206,5 @@
     <origin xyz="0.095 -0.0545 -0.005" rpy="0 0 0"/>
     <geometry>
-      <mesh filename="package://robot_contest/meshes/part13_1.stl" scale="0.001 0.001 0.001"/>
+      <mesh filename="package://spider_robot_description/meshes/part13_1.stl" scale="0.001 0.001 0.001"/>
     </geometry>
   </collision>
@@ -219,5 +219,5 @@
     <origin xyz="0.157173 -0.08008 -0.0304" rpy="0 0 0"/>
     <geometry>
-      <mesh filename="package://robot_contest/meshes/part14_1.stl" scale="0.001 0.001 0.001"/>
+      <mesh filename="package://spider_robot_description/meshes/part14_1.stl" scale="0.001 0.001 0.001"/>
     </geometry>
     <material name="_"/>
@@ -226,5 +226,5 @@
     <origin xyz="0.157173 -0.08008 -0.0304" rpy="0 0 0"/>
     <geometry>
-      <mesh filename="package://robot_contest/meshes/part14_1.stl" scale="0.001 0.001 0.001"/>
+      <mesh filename="package://spider_robot_description/meshes/part14_1.stl" scale="0.001 0.001 0.001"/>
     </geometry>
   </collision>
@@ -239,5 +239,5 @@
     <origin xyz="0.095 0.0545 -0.005" rpy="0 0 0"/>
     <geometry>
-      <mesh filename="package://robot_contest/meshes/part16_1.stl" scale="0.001 0.001 0.001"/>
+      <mesh filename="package://spider_robot_description/meshes/part16_1.stl" scale="0.001 0.001 0.001"/>
     </geometry>
     <material name="_"/>
@@ -246,5 +246,5 @@
     <origin xyz="0.095 0.0545 -0.005" rpy="0 0 0"/>
     <geometry>
-      <mesh filename="package://robot_contest/meshes/part16_1.stl" scale="0.001 0.001 0.001"/>
+      <mesh filename="package://spider_robot_description/meshes/part16_1.stl" scale="0.001 0.001 0.001"/>
     </geometry>
   </collision>
@@ -259,5 +259,5 @@
     <origin xyz="0.157173 0.08008 -0.0304" rpy="0 0 0"/>
     <geometry>
-      <mesh filename="package://robot_contest/meshes/part17_1.stl" scale="0.001 0.001 0.001"/>
+      <mesh filename="package://spider_robot_description/meshes/part17_1.stl" scale="0.001 0.001 0.001"/>
     </geometry>
     <material name="_"/>
@@ -266,5 +266,485 @@
     <origin xyz="0.157173 0.08008 -0.0304" rpy="0 0 0"/>
     <geometry>
-      <mesh filename="package://robot_contest/meshes/part17_1.stl" scale="0.001 0.001 0.001"/>
+      <mesh filename="package://spider_robot_description/meshes/part17_1.stl" scale="0.001 0.001 0.001"/>
+    </geometry>
+  </collision>
+</link>
+<link name="part3_1">
+  <inertial>
+    <origin xyz="0.004221158383464624 -0.04758074361356199 -0.010298255954450997" rpy="0 0 0"/>
+    <mass value="0.12505650813052724"/>
+    <inertia ixx="0.001082" iyy="0.000159" izz="0.001129" ixy="-7.5e-05" iyz="-0.000208" ixz="-1.1e-05"/>
+  </inertial>
+  <visual>
+    <origin xyz="-0.214003 -0.138254 -0.0304" rpy="0 0 0"/>
+    <geometry>
+      <mesh filename="package://spider_robot_description/meshes/part3_1.stl" scale="0.001 0.001 0.001"/>
+    </geometry>
+    <material name="_"/>
+  </visual>
+  <collision>
+    <origin xyz="-0.214003 -0.138254 -0.0304" rpy="0 0 0"/>
+    <geometry>
+      <mesh filename="package://spider_robot_description/meshes/part3_1.stl" scale="0.001 0.001 0.001"/>
+    </geometry>
+  </collision>
+</link>
+<link name="part6_1">
+  <inertial>
+    <origin xyz="0.03479869953680867 0.0592049589644737 -0.010298255954450442" rpy="0 0 0"/>
+    <mass value="0.1250565081305319"/>
+    <inertia ixx="0.001363" iyy="0.000216" izz="0.001467" ixy="-0.000277" iyz="0.000239" ixz="6.3e-05"/>
+  </inertial>
+  <visual>
+    <origin xyz="-0.214003 0.138254 -0.0304" rpy="0 0 0"/>
+    <geometry>
+      <mesh filename="package://spider_robot_description/meshes/part6_1.stl" scale="0.001 0.001 0.001"/>
+    </geometry>
+    <material name="_"/>
+  </visual>
+  <collision>
+    <origin xyz="-0.214003 0.138254 -0.0304" rpy="0 0 0"/>
+    <geometry>
+      <mesh filename="package://spider_robot_description/meshes/part6_1.stl" scale="0.001 0.001 0.001"/>
+    </geometry>
+  </collision>
+</link>
+<link name="part9_1">
+  <inertial>
+    <origin xyz="-0.029793763473125137 0.04613844978067949 -0.010298255954450313" rpy="0 0 0"/>
+    <mass value="0.12505650813053223"/>
+    <inertia ixx="0.000196" iyy="0.000106" izz="0.000191" ixy="-8e-06" iyz="2e-05" ixz="-1.2e-05"/>
+  </inertial>
+  <visual>
+    <origin xyz="-0.024925 -0.197871 -0.0304" rpy="0 0 0"/>
+    <geometry>
+      <mesh filename="package://spider_robot_description/meshes/part9_1.stl" scale="0.001 0.001 0.001"/>
+    </geometry>
+    <material name="_"/>
+  </visual>
+  <collision>
+    <origin xyz="-0.024925 -0.197871 -0.0304" rpy="0 0 0"/>
+    <geometry>
+      <mesh filename="package://spider_robot_description/meshes/part9_1.stl" scale="0.001 0.001 0.001"/>
+    </geometry>
+  </collision>
+</link>
+<link name="part12_1">
+  <inertial>
+    <origin xyz="-0.0763301129730041 -0.06509177558310722 -0.010298255954450247" rpy="0 0 0"/>
+    <mass value="0.12505650813053235"/>
+    <inertia ixx="0.000278" iyy="0.000392" izz="0.000557" ixy="-0.000175" iyz="-6.3e-05" ixz="-0.000111"/>
+  </inertial>
+  <visual>
+    <origin xyz="-0.024925 0.197871 -0.0304" rpy="0 0 0"/>
+    <geometry>
+      <mesh filename="package://spider_robot_description/meshes/part12_1.stl" scale="0.001 0.001 0.001"/>
+    </geometry>
+    <material name="_"/>
+  </visual>
+  <collision>
+    <origin xyz="-0.024925 0.197871 -0.0304" rpy="0 0 0"/>
+    <geometry>
+      <mesh filename="package://spider_robot_description/meshes/part12_1.stl" scale="0.001 0.001 0.001"/>
+    </geometry>
+  </collision>
+</link>
+<link name="part15_1">
+  <inertial>
+    <origin xyz="-0.03721261981245194 0.07321669362063984 -0.010298255954450782" rpy="0 0 0"/>
+    <mass value="0.12505650813052843"/>
+    <inertia ixx="0.000643" iyy="0.000138" izz="0.00067" ixy="-1.1e-05" iyz="0.000146" ixz="1.5e-05"/>
+  </inertial>
+  <visual>
+    <origin xyz="0.178754 -0.173503 -0.0304" rpy="0 0 0"/>
+    <geometry>
+      <mesh filename="package://spider_robot_description/meshes/part15_1.stl" scale="0.001 0.001 0.001"/>
+    </geometry>
+    <material name="_"/>
+  </visual>
+  <collision>
+    <origin xyz="0.178754 -0.173503 -0.0304" rpy="0 0 0"/>
+    <geometry>
+      <mesh filename="package://spider_robot_description/meshes/part15_1.stl" scale="0.001 0.001 0.001"/>
+    </geometry>
+  </collision>
+</link>
+<link name="part18_1">
+  <inertial>
+    <origin xyz="-0.08233230187734139 0.09080916411778589 -0.010298255954450788" rpy="0 0 0"/>
+    <mass value="0.12505650813052913"/>
+    <inertia ixx="0.001224" iyy="0.000322" izz="0.001434" ixy="0.000383" iyz="0.000223" ixz="-8.3e-05"/>
+  </inertial>
+  <visual>
+    <origin xyz="0.178754 0.173503 -0.0304" rpy="0 0 0"/>
+    <geometry>
+      <mesh filename="package://spider_robot_description/meshes/part18_1.stl" scale="0.001 0.001 0.001"/>
+    </geometry>
+    <material name="_"/>
+  </visual>
+  <collision>
+    <origin xyz="0.178754 0.173503 -0.0304" rpy="0 0 0"/>
+    <geometry>
+      <mesh filename="package://spider_robot_description/meshes/part18_1.stl" scale="0.001 0.001 0.001"/>
+    </geometry>
+  </collision>
+</link>
+<link name="d_part1_1">
+  <inertial>
+    <origin xyz="-2.5494084521238136e-07 2.479434127455882e-07 -2.3314683517128287e-15" rpy="0 0 0"/>
+    <mass value="4.110250388446646e-06"/>
+    <inertia ixx="0.0" iyy="0.0" izz="0.0" ixy="0.0" iyz="-0.0" ixz="0.0"/>
+  </inertial>
+  <visual>
+    <origin xyz="-0.294702 -0.255545 -0.0304" rpy="0 0 0"/>
+    <geometry>
+      <mesh filename="package://spider_robot_description/meshes/d_part1_1.stl" scale="0.001 0.001 0.001"/>
+    </geometry>
+    <material name="_"/>
+  </visual>
+  <collision>
+    <origin xyz="-0.294702 -0.255545 -0.0304" rpy="0 0 0"/>
+    <geometry>
+      <mesh filename="package://spider_robot_description/meshes/d_part1_1.stl" scale="0.001 0.001 0.001"/>
+    </geometry>
+  </collision>
+</link>
+<link name="d_part2_1">
+  <inertial>
+    <origin xyz="-2.5494084521238136e-07 2.479434127455882e-07 -2.3314683517128287e-15" rpy="0 0 0"/>
+    <mass value="4.110250388446646e-06"/>
+    <inertia ixx="0.0" iyy="0.0" izz="0.0" ixy="0.0" iyz="-0.0" ixz="0.0"/>
+  </inertial>
+  <visual>
+    <origin xyz="-0.294702 -0.255545 -0.0304" rpy="0 0 0"/>
+    <geometry>
+      <mesh filename="package://spider_robot_description/meshes/d_part2_1.stl" scale="0.001 0.001 0.001"/>
+    </geometry>
+    <material name="_"/>
+  </visual>
+  <collision>
+    <origin xyz="-0.294702 -0.255545 -0.0304" rpy="0 0 0"/>
+    <geometry>
+      <mesh filename="package://spider_robot_description/meshes/d_part2_1.stl" scale="0.001 0.001 0.001"/>
+    </geometry>
+  </collision>
+</link>
+<link name="d_part3_1">
+  <inertial>
+    <origin xyz="-2.5494084521238136e-07 2.479434127455882e-07 -2.3314683517128287e-15" rpy="0 0 0"/>
+    <mass value="4.110250388446646e-06"/>
+    <inertia ixx="0.0" iyy="0.0" izz="0.0" ixy="0.0" iyz="-0.0" ixz="0.0"/>
+  </inertial>
+  <visual>
+    <origin xyz="-0.294702 -0.255545 -0.0304" rpy="0 0 0"/>
+    <geometry>
+      <mesh filename="package://spider_robot_description/meshes/d_part3_1.stl" scale="0.001 0.001 0.001"/>
+    </geometry>
+    <material name="_"/>
+  </visual>
+  <collision>
+    <origin xyz="-0.294702 -0.255545 -0.0304" rpy="0 0 0"/>
+    <geometry>
+      <mesh filename="package://spider_robot_description/meshes/d_part3_1.stl" scale="0.001 0.001 0.001"/>
+    </geometry>
+  </collision>
+</link>
+<link name="d_part4_1">
+  <inertial>
+    <origin xyz="-2.5494084748833856e-07 -2.4794341335621084e-07 -2.321060010856968e-15" rpy="0 0 0"/>
+    <mass value="4.110250388446646e-06"/>
+    <inertia ixx="0.0" iyy="0.0" izz="0.0" ixy="0.0" iyz="0.0" ixz="0.0"/>
+  </inertial>
+  <visual>
+    <origin xyz="-0.294702 0.255545 -0.0304" rpy="0 0 0"/>
+    <geometry>
+      <mesh filename="package://spider_robot_description/meshes/d_part4_1.stl" scale="0.001 0.001 0.001"/>
+    </geometry>
+    <material name="_"/>
+  </visual>
+  <collision>
+    <origin xyz="-0.294702 0.255545 -0.0304" rpy="0 0 0"/>
+    <geometry>
+      <mesh filename="package://spider_robot_description/meshes/d_part4_1.stl" scale="0.001 0.001 0.001"/>
+    </geometry>
+  </collision>
+</link>
+<link name="d_part5_1">
+  <inertial>
+    <origin xyz="-2.5494084748833856e-07 -2.4794341335621084e-07 -2.321060010856968e-15" rpy="0 0 0"/>
+    <mass value="4.110250388446646e-06"/>
+    <inertia ixx="0.0" iyy="0.0" izz="0.0" ixy="0.0" iyz="0.0" ixz="0.0"/>
+  </inertial>
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