Commit message: fix model

File: urdf/spider_robot.xacro (robot description, xacro)
@@ -1,7 +1,7 @@
 <?xml version="1.0" ?>
 <robot name="spider_robot" xmlns:xacro="http://www.ros.org/wiki/xacro">
-<xacro:include filename="$(find spider_robot_description)/urdf/materials.xacro" />
-<xacro:include filename="$(find spider_robot_description)/urdf/spider_robot.trans" />
-<xacro:include filename="$(find spider_robot_description)/urdf/spider_robot.gazebo" />
+<xacro:include filename="$(find robot_contest)/urdf/materials.xacro" />
+<xacro:include filename="$(find robot_contest)/urdf/spider_robot.trans" />
+<xacro:include filename="$(find robot_contest)/urdf/spider_robot.gazebo" />
 <link name="dummy">
 </link>
@@ -19,5 +19,5 @@
     <origin xyz="0 0 0" rpy="0 0 0"/>
     <geometry>
-      <mesh filename="package://spider_robot_description/meshes/base_link.stl" scale="0.001 0.001 0.001"/>
+      <mesh filename="package://robot_contest/meshes/base_link.stl" scale="0.001 0.001 0.001"/>
     </geometry>
     <material name="_"/>
@@ -26,5 +26,5 @@
     <origin xyz="0 0 0" rpy="0 0 0"/>
     <geometry>
-      <mesh filename="package://spider_robot_description/meshes/base_link.stl" scale="0.001 0.001 0.001"/>
+      <mesh filename="package://robot_contest/meshes/base_link.stl" scale="0.001 0.001 0.001"/>
     </geometry>
   </collision>
@@ -39,5 +39,5 @@
     <origin xyz="-0.095 -0.0545 -0.005" rpy="0 0 0"/>
     <geometry>
-      <mesh filename="package://spider_robot_description/meshes/part1_1.stl" scale="0.001 0.001 0.001"/>
+      <mesh filename="package://robot_contest/meshes/part1_1.stl" scale="0.001 0.001 0.001"/>
     </geometry>
     <material name="_"/>
@@ -46,5 +46,5 @@
     <origin xyz="-0.095 -0.0545 -0.005" rpy="0 0 0"/>
     <geometry>
-      <mesh filename="package://spider_robot_description/meshes/part1_1.stl" scale="0.001 0.001 0.001"/>
+      <mesh filename="package://robot_contest/meshes/part1_1.stl" scale="0.001 0.001 0.001"/>
     </geometry>
   </collision>
@@ -59,5 +59,5 @@
     <origin xyz="-0.12058 -0.116673 -0.0304" rpy="0 0 0"/>
     <geometry>
-      <mesh filename="package://spider_robot_description/meshes/part2_1.stl" scale="0.001 0.001 0.001"/>
+      <mesh filename="package://robot_contest/meshes/part2_1.stl" scale="0.001 0.001 0.001"/>
     </geometry>
     <material name="_"/>
@@ -66,5 +66,5 @@
     <origin xyz="-0.12058 -0.116673 -0.0304" rpy="0 0 0"/>
     <geometry>
-      <mesh filename="package://spider_robot_description/meshes/part2_1.stl" scale="0.001 0.001 0.001"/>
+      <mesh filename="package://robot_contest/meshes/part2_1.stl" scale="0.001 0.001 0.001"/>
     </geometry>
   </collision>
@@ -79,5 +79,5 @@
     <origin xyz="-0.095 0.0545 -0.005" rpy="0 0 0"/>
     <geometry>
-      <mesh filename="package://spider_robot_description/meshes/part4_1.stl" scale="0.001 0.001 0.001"/>
+      <mesh filename="package://robot_contest/meshes/part4_1.stl" scale="0.001 0.001 0.001"/>
     </geometry>
     <material name="_"/>
@@ -86,5 +86,5 @@
     <origin xyz="-0.095 0.0545 -0.005" rpy="0 0 0"/>
     <geometry>
-      <mesh filename="package://spider_robot_description/meshes/part4_1.stl" scale="0.001 0.001 0.001"/>
+      <mesh filename="package://robot_contest/meshes/part4_1.stl" scale="0.001 0.001 0.001"/>
     </geometry>
   </collision>
@@ -99,5 +99,5 @@
     <origin xyz="-0.12058 0.116673 -0.0304" rpy="0 0 0"/>
     <geometry>
-      <mesh filename="package://spider_robot_description/meshes/part5_1.stl" scale="0.001 0.001 0.001"/>
+      <mesh filename="package://robot_contest/meshes/part5_1.stl" scale="0.001 0.001 0.001"/>
     </geometry>
     <material name="_"/>
@@ -106,5 +106,5 @@
     <origin xyz="-0.12058 0.116673 -0.0304" rpy="0 0 0"/>
     <geometry>
-      <mesh filename="package://spider_robot_description/meshes/part5_1.stl" scale="0.001 0.001 0.001"/>
+      <mesh filename="package://robot_contest/meshes/part5_1.stl" scale="0.001 0.001 0.001"/>
     </geometry>
   </collision>
@@ -119,5 +119,5 @@
     <origin xyz="-0.0 -0.0545 -0.005" rpy="0 0 0"/>
     <geometry>
-      <mesh filename="package://spider_robot_description/meshes/part7_1.stl" scale="0.001 0.001 0.001"/>
+      <mesh filename="package://robot_contest/meshes/part7_1.stl" scale="0.001 0.001 0.001"/>
     </geometry>
     <material name="_"/>
@@ -126,5 +126,5 @@
     <origin xyz="-0.0 -0.0545 -0.005" rpy="0 0 0"/>
     <geometry>
-      <mesh filename="package://spider_robot_description/meshes/part7_1.stl" scale="0.001 0.001 0.001"/>
+      <mesh filename="package://robot_contest/meshes/part7_1.stl" scale="0.001 0.001 0.001"/>
     </geometry>
   </collision>
@@ -139,5 +139,5 @@
     <origin xyz="0.025875 -0.116551 -0.0304" rpy="0 0 0"/>
     <geometry>
-      <mesh filename="package://spider_robot_description/meshes/part8_1.stl" scale="0.001 0.001 0.001"/>
+      <mesh filename="package://robot_contest/meshes/part8_1.stl" scale="0.001 0.001 0.001"/>
     </geometry>
     <material name="_"/>
@@ -146,5 +146,5 @@
     <origin xyz="0.025875 -0.116551 -0.0304" rpy="0 0 0"/>
     <geometry>
-      <mesh filename="package://spider_robot_description/meshes/part8_1.stl" scale="0.001 0.001 0.001"/>
+      <mesh filename="package://robot_contest/meshes/part8_1.stl" scale="0.001 0.001 0.001"/>
     </geometry>
   </collision>
@@ -159,5 +159,5 @@
     <origin xyz="0.0 0.0545 -0.005" rpy="0 0 0"/>
     <geometry>
-      <mesh filename="package://spider_robot_description/meshes/part10_1.stl" scale="0.001 0.001 0.001"/>
+      <mesh filename="package://robot_contest/meshes/part10_1.stl" scale="0.001 0.001 0.001"/>
     </geometry>
     <material name="_"/>
@@ -166,5 +166,5 @@
     <origin xyz="0.0 0.0545 -0.005" rpy="0 0 0"/>
     <geometry>
-      <mesh filename="package://spider_robot_description/meshes/part10_1.stl" scale="0.001 0.001 0.001"/>
+      <mesh filename="package://robot_contest/meshes/part10_1.stl" scale="0.001 0.001 0.001"/>
     </geometry>
   </collision>
@@ -179,5 +179,5 @@
     <origin xyz="0.025875 0.116551 -0.0304" rpy="0 0 0"/>
     <geometry>
-      <mesh filename="package://spider_robot_description/meshes/part11_1.stl" scale="0.001 0.001 0.001"/>
+      <mesh filename="package://robot_contest/meshes/part11_1.stl" scale="0.001 0.001 0.001"/>
     </geometry>
     <material name="_"/>
@@ -186,5 +186,5 @@
     <origin xyz="0.025875 0.116551 -0.0304" rpy="0 0 0"/>
     <geometry>
-      <mesh filename="package://spider_robot_description/meshes/part11_1.stl" scale="0.001 0.001 0.001"/>
+      <mesh filename="package://robot_contest/meshes/part11_1.stl" scale="0.001 0.001 0.001"/>
     </geometry>
   </collision>
@@ -199,5 +199,5 @@
     <origin xyz="0.095 -0.0545 -0.005" rpy="0 0 0"/>
     <geometry>
-      <mesh filename="package://spider_robot_description/meshes/part13_1.stl" scale="0.001 0.001 0.001"/>
+      <mesh filename="package://robot_contest/meshes/part13_1.stl" scale="0.001 0.001 0.001"/>
     </geometry>
     <material name="_"/>
@@ -206,5 +206,5 @@
     <origin xyz="0.095 -0.0545 -0.005" rpy="0 0 0"/>
     <geometry>
-      <mesh filename="package://spider_robot_description/meshes/part13_1.stl" scale="0.001 0.001 0.001"/>
+      <mesh filename="package://robot_contest/meshes/part13_1.stl" scale="0.001 0.001 0.001"/>
     </geometry>
   </collision>
@@ -219,5 +219,5 @@
     <origin xyz="0.157173 -0.08008 -0.0304" rpy="0 0 0"/>
     <geometry>
-      <mesh filename="package://spider_robot_description/meshes/part14_1.stl" scale="0.001 0.001 0.001"/>
+      <mesh filename="package://robot_contest/meshes/part14_1.stl" scale="0.001 0.001 0.001"/>
     </geometry>
     <material name="_"/>
@@ -226,5 +226,5 @@
     <origin xyz="0.157173 -0.08008 -0.0304" rpy="0 0 0"/>
     <geometry>
-      <mesh filename="package://spider_robot_description/meshes/part14_1.stl" scale="0.001 0.001 0.001"/>
+      <mesh filename="package://robot_contest/meshes/part14_1.stl" scale="0.001 0.001 0.001"/>
     </geometry>
   </collision>
@@ -239,5 +239,5 @@
     <origin xyz="0.095 0.0545 -0.005" rpy="0 0 0"/>
     <geometry>
-      <mesh filename="package://spider_robot_description/meshes/part16_1.stl" scale="0.001 0.001 0.001"/>
+      <mesh filename="package://robot_contest/meshes/part16_1.stl" scale="0.001 0.001 0.001"/>
     </geometry>
     <material name="_"/>
@@ -246,5 +246,5 @@
     <origin xyz="0.095 0.0545 -0.005" rpy="0 0 0"/>
     <geometry>
-      <mesh filename="package://spider_robot_description/meshes/part16_1.stl" scale="0.001 0.001 0.001"/>
+      <mesh filename="package://robot_contest/meshes/part16_1.stl" scale="0.001 0.001 0.001"/>
     </geometry>
   </collision>
@@ -259,5 +259,5 @@
     <origin xyz="0.157173 0.08008 -0.0304" rpy="0 0 0"/>
     <geometry>
-      <mesh filename="package://spider_robot_description/meshes/part17_1.stl" scale="0.001 0.001 0.001"/>
+      <mesh filename="package://robot_contest/meshes/part17_1.stl" scale="0.001 0.001 0.001"/>
     </geometry>
     <material name="_"/>
@@ -266,5 +266,5 @@
     <origin xyz="0.157173 0.08008 -0.0304" rpy="0 0 0"/>
     <geometry>
-      <mesh filename="package://spider_robot_description/meshes/part17_1.stl" scale="0.001 0.001 0.001"/>
+      <mesh filename="package://robot_contest/meshes/part17_1.stl" scale="0.001 0.001 0.001"/>
     </geometry>
   </collision>
@@ -279,5 +279,5 @@
     <origin xyz="-0.214003 -0.138254 -0.0304" rpy="0 0 0"/>
     <geometry>
-      <mesh filename="package://spider_robot_description/meshes/part3_1.stl" scale="0.001 0.001 0.001"/>
+      <mesh filename="package://robot_contest/meshes/part3_1.stl" scale="0.001 0.001 0.001"/>
     </geometry>
     <material name="_"/>
@@ -286,5 +286,5 @@
     <origin xyz="-0.214003 -0.138254 -0.0304" rpy="0 0 0"/>
     <geometry>
-      <mesh filename="package://spider_robot_description/meshes/part3_1.stl" scale="0.001 0.001 0.001"/>
+      <mesh filename="package://robot_contest/meshes/part3_1.stl" scale="0.001 0.001 0.001"/>
     </geometry>
   </collision>
@@ -299,5 +299,5 @@
     <origin xyz="-0.214003 0.138254 -0.0304" rpy="0 0 0"/>
     <geometry>
-      <mesh filename="package://spider_robot_description/meshes/part6_1.stl" scale="0.001 0.001 0.001"/>
+      <mesh filename="package://robot_contest/meshes/part6_1.stl" scale="0.001 0.001 0.001"/>
     </geometry>
     <material name="_"/>
@@ -306,5 +306,5 @@
     <origin xyz="-0.214003 0.138254 -0.0304" rpy="0 0 0"/>
     <geometry>
-      <mesh filename="package://spider_robot_description/meshes/part6_1.stl" scale="0.001 0.001 0.001"/>
+      <mesh filename="package://robot_contest/meshes/part6_1.stl" scale="0.001 0.001 0.001"/>
     </geometry>
   </collision>
@@ -319,5 +319,5 @@
     <origin xyz="-0.024925 -0.197871 -0.0304" rpy="0 0 0"/>
     <geometry>
-      <mesh filename="package://spider_robot_description/meshes/part9_1.stl" scale="0.001 0.001 0.001"/>
+      <mesh filename="package://robot_contest/meshes/part9_1.stl" scale="0.001 0.001 0.001"/>
     </geometry>
     <material name="_"/>
@@ -326,5 +326,5 @@
     <origin xyz="-0.024925 -0.197871 -0.0304" rpy="0 0 0"/>
     <geometry>
-      <mesh filename="package://spider_robot_description/meshes/part9_1.stl" scale="0.001 0.001 0.001"/>
+      <mesh filename="package://robot_contest/meshes/part9_1.stl" scale="0.001 0.001 0.001"/>
     </geometry>
   </collision>
@@ -339,5 +339,5 @@
     <origin xyz="-0.024925 0.197871 -0.0304" rpy="0 0 0"/>
     <geometry>
-      <mesh filename="package://spider_robot_description/meshes/part12_1.stl" scale="0.001 0.001 0.001"/>
+      <mesh filename="package://robot_contest/meshes/part12_1.stl" scale="0.001 0.001 0.001"/>
     </geometry>
     <material name="_"/>
@@ -346,5 +346,5 @@
     <origin xyz="-0.024925 0.197871 -0.0304" rpy="0 0 0"/>
     <geometry>
-      <mesh filename="package://spider_robot_description/meshes/part12_1.stl" scale="0.001 0.001 0.001"/>
+      <mesh filename="package://robot_contest/meshes/part12_1.stl" scale="0.001 0.001 0.001"/>
     </geometry>
   </collision>
@@ -359,5 +359,5 @@
     <origin xyz="0.178754 -0.173503 -0.0304" rpy="0 0 0"/>
     <geometry>
-      <mesh filename="package://spider_robot_description/meshes/part15_1.stl" scale="0.001 0.001 0.001"/>
+      <mesh filename="package://robot_contest/meshes/part15_1.stl" scale="0.001 0.001 0.001"/>
     </geometry>
     <material name="_"/>
@@ -366,5 +366,5 @@
     <origin xyz="0.178754 -0.173503 -0.0304" rpy="0 0 0"/>
     <geometry>
-      <mesh filename="package://spider_robot_description/meshes/part15_1.stl" scale="0.001 0.001 0.001"/>
+      <mesh filename="package://robot_contest/meshes/part15_1.stl" scale="0.001 0.001 0.001"/>
     </geometry>
   </collision>
@@ -379,5 +379,5 @@
     <origin xyz="0.178754 0.173503 -0.0304" rpy="0 0 0"/>
     <geometry>
-      <mesh filename="package://spider_robot_description/meshes/part18_1.stl" scale="0.001 0.001 0.001"/>
+      <mesh filename="package://robot_contest/meshes/part18_1.stl" scale="0.001 0.001 0.001"/>
     </geometry>
     <material name="_"/>
@@ -386,5 +386,5 @@
     <origin xyz="0.178754 0.173503 -0.0304" rpy="0 0 0"/>
     <geometry>
-      <mesh filename="package://spider_robot_description/meshes/part18_1.stl" scale="0.001 0.001 0.001"/>
+      <mesh filename="package://robot_contest/meshes/part18_1.stl" scale="0.001 0.001 0.001"/>
     </geometry>
   </collision>
@@ -399,5 +399,5 @@
     <origin xyz="-0.294702 -0.255545 -0.0304" rpy="0 0 0"/>
     <geometry>
-      <mesh filename="package://spider_robot_description/meshes/d_part1_1.stl" scale="0.001 0.001 0.001"/>
+      <mesh filename="package://robot_contest/meshes/d_part1_1.stl" scale="0.001 0.001 0.001"/>
     </geometry>
     <material name="_"/>
@@ -406,5 +406,5 @@
     <origin xyz="-0.294702 -0.255545 -0.0304" rpy="0 0 0"/>
     <geometry>
-      <mesh filename="package://spider_robot_description/meshes/d_part1_1.stl" scale="0.001 0.001 0.001"/>
+      <mesh filename="package://robot_contest/meshes/d_part1_1.stl" scale="0.001 0.001 0.001"/>
     </geometry>
   </collision>
@@ -419,5 +419,5 @@
     <origin xyz="-0.294702 -0.255545 -0.0304" rpy="0 0 0"/>
     <geometry>
-      <mesh filename="package://spider_robot_description/meshes/d_part2_1.stl" scale="0.001 0.001 0.001"/>
+      <mesh filename="package://robot_contest/meshes/d_part2_1.stl" scale="0.001 0.001 0.001"/>
     </geometry>
     <material name="_"/>
@@ -426,5 +426,5 @@
     <origin xyz="-0.294702 -0.255545 -0.0304" rpy="0 0 0"/>
     <geometry>
-      <mesh filename="package://spider_robot_description/meshes/d_part2_1.stl" scale="0.001 0.001 0.001"/>
+      <mesh filename="package://robot_contest/meshes/d_part2_1.stl" scale="0.001 0.001 0.001"/>
     </geometry>
   </collision>
@@ -439,5 +439,5 @@
     <origin xyz="-0.294702 -0.255545 -0.0304" rpy="0 0 0"/>
     <geometry>
-      <mesh filename="package://spider_robot_description/meshes/d_part3_1.stl" scale="0.001 0.001 0.001"/>
+      <mesh filename="package://robot_contest/meshes/d_part3_1.stl" scale="0.001 0.001 0.001"/>
     </geometry>
     <material name="_"/>
@@ -446,5 +446,5 @@
     <origin xyz="-0.294702 -0.255545 -0.0304" rpy="0 0 0"/>
     <geometry>
-      <mesh filename="package://spider_robot_description/meshes/d_part3_1.stl" scale="0.001 0.001 0.001"/>
+      <mesh filename="package://robot_contest/meshes/d_part3_1.stl" scale="0.001 0.001 0.001"/>
     </geometry>
   </collision>
@@ -459,5 +459,5 @@
     <origin xyz="-0.294702 0.255545 -0.0304" rpy="0 0 0"/>
     <geometry>
-      <mesh filename="package://spider_robot_description/meshes/d_part4_1.stl" scale="0.001 0.001 0.001"/>
+      <mesh filename="package://robot_contest/meshes/d_part4_1.stl" scale="0.001 0.001 0.001"/>
     </geometry>
     <material name="_"/>
@@ -466,5 +466,5 @@
     <origin xyz="-0.294702 0.255545 -0.0304" rpy="0 0 0"/>
     <geometry>
-      <mesh filename="package://spider_robot_description/meshes/d_part4_1.stl" scale="0.001 0.001 0.001"/>
+      <mesh filename="package://robot_contest/meshes/d_part4_1.stl" scale="0.001 0.001 0.001"/>
     </geometry>
   </collision>
@@ -479,5 +479,5 @@
     <origin xyz="-0.294702 0.255545 -0.0304" rpy="0 0 0"/>
     <geometry>
-      <mesh filename="package://spider_robot_description/meshes/d_part5_1.stl" scale="0.001 0.001 0.001"/>
+      <mesh filename="package://robot_contest/meshes/d_part5_1.stl" scale="0.001 0.001 0.001"/>
     </geometry>
     <material name="_"/>
@@ -486,5 +486,5 @@
     <origin xyz="-0.294702 0.255545 -0.0304" rpy="0 0 0"/>
     <geometry>
-      <mesh filename="package://spider_robot_description/meshes/d_part5_1.stl" scale="0.001 0.001 0.001"/>
+      <mesh filename="package://robot_contest/meshes/d_part5_1.stl" scale="0.001 0.001 0.001"/>
     </geometry>
   </collision>
@@ -499,5 +499,5 @@
     <origin xyz="-0.294702 0.255545 -0.0304" rpy="0 0 0"/>
     <geometry>
-      <mesh filename="package://spider_robot_description/meshes/d_part6_1.stl" scale="0.001 0.001 0.001"/>
+      <mesh filename="package://robot_contest/meshes/d_part6_1.stl" scale="0.001 0.001 0.001"/>
     </geometry>
     <material name="_"/>
@@ -506,5 +506,5 @@
     <origin xyz="-0.294702 0.255545 -0.0304" rpy="0 0 0"/>
     <geometry>
-      <mesh filename="package://spider_robot_description/meshes/d_part6_1.stl" scale="0.001 0.001 0.001"/>
+      <mesh filename="package://robot_contest/meshes/d_part6_1.stl" scale="0.001 0.001 0.001"/>
     </geometry>
   </collision>
@@ -519,5 +519,5 @@
     <origin xyz="0.00095 -0.337871 -0.0304" rpy="0 0 0"/>
     <geometry>
-      <mesh filename="package://spider_robot_description/meshes/d_part7_1.stl" scale="0.001 0.001 0.001"/>
+      <mesh filename="package://robot_contest/meshes/d_part7_1.stl" scale="0.001 0.001 0.001"/>
     </geometry>
     <material name="_"/>
@@ -526,5 +526,5 @@
     <origin xyz="0.00095 -0.337871 -0.0304" rpy="0 0 0"/>
     <geometry>
-      <mesh filename="package://spider_robot_description/meshes/d_part7_1.stl" scale="0.001 0.001 0.001"/>
+      <mesh filename="package://robot_contest/meshes/d_part7_1.stl" scale="0.001 0.001 0.001"/>
     </geometry>
   </collision>
@@ -539,5 +539,5 @@
     <origin xyz="0.00095 -0.337871 -0.0304" rpy="0 0 0"/>
     <geometry>
-      <mesh filename="package://spider_robot_description/meshes/d_part8_1.stl" scale="0.001 0.001 0.001"/>
+      <mesh filename="package://robot_contest/meshes/d_part8_1.stl" scale="0.001 0.001 0.001"/>
     </geometry>
     <material name="_"/>
@@ -546,5 +546,5 @@
     <origin xyz="0.00095 -0.337871 -0.0304" rpy="0 0 0"/>
     <geometry>
-      <mesh filename="package://spider_robot_description/meshes/d_part8_1.stl" scale="0.001 0.001 0.001"/>
+      <mesh filename="package://robot_contest/meshes/d_part8_1.stl" scale="0.001 0.001 0.001"/>
     </geometry>
   </collision>
@@ -559,5 +559,5 @@
     <origin xyz="0.00095 -0.337871 -0.0304" rpy="0 0 0"/>
     <geometry>
-      <mesh filename="package://spider_robot_description/meshes/d_part9_1.stl" scale="0.001 0.001 0.001"/>
+      <mesh filename="package://robot_contest/meshes/d_part9_1.stl" scale="0.001 0.001 0.001"/>
     </geometry>
     <material name="_"/>
@@ -566,5 +566,5 @@
     <origin xyz="0.00095 -0.337871 -0.0304" rpy="0 0 0"/>
     <geometry>
-      <mesh filename="package://spider_robot_description/meshes/d_part9_1.stl" scale="0.001 0.001 0.001"/>
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
Commit message: fix model

File: urdf/spider_robot.xacro (robot description, xacro)
@@ -976,5 +976,5 @@
 <joint name="d_rev17" type="continuous">
   <origin xyz="0.0 0.0 0.0" rpy="0 0 0"/>
-  <parent link="part18_1"/>
+  <parent link="d_part16_1"/>
   <child link="d_part17_1"/>
   <axis xyz="-0.707107 0.707107 0.0"/>
@@ -982,5 +982,5 @@
 <joint name="d_rev18" type="continuous">
   <origin xyz="0.0 0.0 0.0" rpy="0 0 0"/>
-  <parent link="part18_1"/>
+  <parent link="d_part17_1"/>
   <child link="d_part18_1"/>
   <axis xyz="-0.0 -0.0 1.0"/>
